File: Untitled.sch (KiCad schematic (older format))
At the start: 20 parts, among them J1 JAMMA, J2 TEST_SW, J3 PLAYER1, J4 PLAYER2, J5 PWR_IN, J6 DC2DC, J7 SCART-F

Commit message: ESP32, shift register and buffer
Parts:
- removed J2: TEST_SW, Buttons_Switches_THT:SW_PUSH_6mm, symbol CONN_02X01
- removed J3: PLAYER1, Connectors:DB15MD, symbol DB15_FEMALE_MountingHoles
- removed J4: PLAYER2, Connectors:DB15MD, symbol DB15_FEMALE_MountingHoles
- added C4: 1u, Capacitors_SMD:C_1206_HandSoldering, symbol C
- added J2: CONN_01X06, Pin_Headers:Pin_Header_Straight_1x06, symbol CONN_01X06
- added U1: LD1117S33TR, TO_SOT_Packages_SMD:SOT-223, symbol LD1117S33TR
- added U2: ESP32-WROOM, ESP32-footprints-Lib:ESP32-WROOM, symbol ESP32-WROOM
- added U3, U4, U5: 74HC595, Housings_SOIC:SOIC-16_3.9x9.9mm_Pitch1.27mm, symbol 74HC595
- added U6, U7, U8, U9: 74LS06, Housings_SOIC:SOIC-14_3.9x8.7mm_Pitch1.27mm_HandSoldering, symbol 74LS06
Connections:
- net labels added: 33, CLK, CLR, DATA, EN, LATCH, OE, VCC
- wire segments 56 -> 151
- no-connect marks 26 -> 47
Other:
- moved on the sheet: C1, C2, C3, J5, J6, J7, R1, R10, R2, R3, R4, R5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

Commit message: Changed over to NPN transistors as driver
Parts:
- removed U6, U7, U8, U9: 74LS06, Housings_SOIC:SOIC-14_3.9x8.7mm_Pitch1.27mm_HandSoldering, symbol 74LS06
- added Q1, Q10, Q11, Q12, Q13, Q14, Q15, Q16, Q17, Q18, Q19, Q2, Q20, Q21, Q22, Q3, Q4, Q5, Q6, Q7, Q8, Q9: Q_NPN_BEC, TO_SOT_Packages_SMD:SOT-23_Handsoldering, symbol Q_NPN_BEC
- added R11, R12, R13, R14, R15, R16, R17, R18, R19, R20, R21, R22, R23, R24, R25, R26, R27, R28, R29, R30, R31, R32: R, Resistors_SMD:R_1206_HandSoldering, symbol R
Connections:
- net +5V: no longer U3.16 (VCC), U4.16 (VCC), U5.16 (VCC)
- net A1: now also Q5.3 (C)
- net A2: now also Q10.3 (C)
- net B1: now also Q16.3 (C)
- net B2: now also Q21.3 (C)
- net C1: now also Q6.3 (C)
- net C2: now also Q11.3 (C)
- net CLR: now also U2.31 (IO19); no longer U2.29 (IO5)
- net COIN1: now also Q2.3 (C)
- net COIN2: now also Q7.3 (C)
- net D1: now also Q17.3 (C)
- net D2: now also Q22.3 (C)
- net DATA: now also U2.27 (IO16); no longer U2.31 (IO19)
- net DOWN1: now also Q14.3 (C)
- net DOWN2: now also Q19.3 (C)
- net GND: now also Q1.2 (E), Q10.2 (E), Q11.2 (E), Q12.2 (E), Q13.2 (E), Q14.2 (E), Q15.2 (E), Q16.2 (E), Q17.2 (E), Q18.2 (E), Q19.2 (E), Q2.2 (E), Q20.2 (E), Q21.2 (E), Q22.2 (E), Q3.2 (E), Q4.2 (E), Q5.2 (E), Q6.2 (E), Q7.2 (E), Q8.2 (E), Q9.2 (E)
- net LATCH: now also U2.29 (IO5); no longer U2.28 (IO17)
- net LEFT1: now also Q4.3 (C)
- net LEFT2: now also Q9.3 (C)
- net OE: now also U2.28 (IO17); no longer U2.27 (IO16)
- net RIGHT1: now also Q15.3 (C)
- net RIGHT2: now also Q20.3 (C)
- net SERVICE: now also Q12.3 (C)
- net START1: now also Q13.3 (C)
- net START2: now also Q18.3 (C)
- net TEST: now also Q1.3 (C)
- net UP1: now also Q3.3 (C)
- net UP2: now also Q8.3 (C)
- net at U3.15 (QA): now also R11.2
- net at U3.1 (QB): now also R12.2
- net at U3.2 (QC): now also R13.2
- net at U3.3 (QD): now also R14.2
- net at U3.4 (QE): now also R15.2
- net at U3.5 (QF): now also R16.2
- net at U3.6 (QG): now also R17.2
- net at U3.7 (QH): now also R18.2
- net at U4.15 (QA): now also R19.2
- net at U4.1 (QB): now also R20.2
- net at U4.2 (QC): now also R21.2
- net at U4.3 (QD): now also R22.2
- net at U4.4 (QE): now also R23.2
- net at U4.5 (QF): now also R24.2
- net at U4.6 (QG): now also R25.2
- net at U4.7 (QH): now also R26.2
- net at U5.15 (QA): now also R27.2
- net at U5.1 (QB): now also R28.2
- net at U5.2 (QC): now also R29.2
- net at U5.3 (QD): now also R30.2
- net at U5.4 (QE): now also R31.2
- net at U5.5 (QF): now also R32.2
- net 33 renamed VCC
- net VCC: now also U3.16 (VCC), U4.16 (VCC), U5.16 (VCC)
- new net: Q2.1 (B), R13.1
- new net: Q13.1 (B), R14.1
- new net: Q1.1 (B), R11.1
- new net: Q12.1 (B), R12.1
- new net: Q4.1 (B), R17.1
- new net: Q15.1 (B), R18.1
- new net: Q3.1 (B), R15.1
- new net: Q14.1 (B), R16.1
- new net: Q6.1 (B), R21.1
- new net: Q17.1 (B), R22.1
- new net: Q5.1 (B), R19.1
- new net: Q16.1 (B), R20.1
- new net: Q8.1 (B), R25.1
- new net: Q19.1 (B), R26.1
- new net: Q7.1 (B), R23.1
- new net: Q18.1 (B), R24.1
- new net: Q10.1 (B), R29.1
- new net: Q21.1 (B), R30.1
- new net: Q9.1 (B), R27.1
- new net: Q20.1 (B), R28.1
- new net: Q11.1 (B), R31.1
- new net: Q22.1 (B), R32.1

Commit message: Simplied version using LED driver chips
Parts:
- removed Q1, Q10, Q11, Q12, Q13, Q14, Q15, Q16, Q17, Q18, Q19, Q2, Q20, Q21, Q22, Q3, Q4, Q5, Q6, Q7, Q8, Q9: Q_NPN_BEC, TO_SOT_Packages_SMD:SOT-23_Handsoldering, symbol Q_NPN_BEC
- removed R13, R14, R15, R16, R17, R18, R19, R20, R21, R22, R23, R24, R25, R26, R27, R28, R29, R30, R31, R32: R, Resistors_SMD:R_1206_HandSoldering, symbol R
- removed U3, U4, U5: 74HC595, Housings_SOIC:SOIC-16_3.9x9.9mm_Pitch1.27mm, symbol 74HC595
- added U3, U4: TLC5926IDW, Housings_SOIC:SOIC-24W_7.5x15.4mm_Pitch1.27mm, symbol TLC5926IDW
Connections:
- net A1: now also U3.8 (OUT3)
- net A2: now also U4.17 (OUT12)
- net B1: now also U3.7 (OUT2)
- net B2: now also U4.18 (OUT13)
- net C1: now also U3.6 (OUT1)
- net C2: now also U4.19 (OUT14)
- net CLK: now also U3.3 (CLK), U4.3 (CLK)
- net COIN1: now also U3.14 (OUT9)
- net COIN2: now also U4.11 (OUT6)
- net D1: now also U3.5 (OUT0)
- net D2: now also U4.20 (OUT15)
- net DATA: now also U3.2 (SDI)
- net DOWN1: now also U3.11 (OUT6)
- net DOWN2: now also U4.14 (OUT9)
- net GND: now also R11.2, R12.2, U3.1 (GND), U4.1 (GND)
- net LATCH: now also U3.4 (LE(ED1)), U4.4 (LE(ED1))
- net LEFT1: now also U3.10 (OUT5)
- net LEFT2: now also U4.15 (OUT10)
- net OE: now also U3.21 (~OE~(ED2)), U4.21 (~OE~(ED2))
- net RIGHT1: now also U3.9 (OUT4)
- net RIGHT2: now also U4.16 (OUT11)
- net SERVICE: now also U4.12 (OUT7)
- net START1: now also U3.15 (OUT10)
- net START2: now also U4.10 (OUT5)
- net TEST: now also U3.13 (OUT8)
- net UP1: now also U3.12 (OUT7)
- net UP2: now also U4.13 (OUT8)
- net VCC: now also U3.24 (V+), U4.24 (V+)
- net at R11.1: now also U3.23 (REXT)
- net at R12.1: now also U4.23 (REXT)
- new net: U3.22 (SDO), U4.2 (SDI)
- no-connect marks 47 -> 55

Commit message: Added reset/upload buttons
Parts:
- added SW1, SW2, SW3: SW_Push, Buttons_Switches_SMD:SW_SPST_EVQPE1, symbol SW_Push
Connections:
- net GND: now also SW1.2, SW2.1, SW3.2
- net VCC: now also J2.4 (P4); no longer J2.5 (P5)
- net at J6.1 (P1): now also SW1.1
- net at U2.25 (IO0): now also SW3.1; no longer J2.3 (P3)
- net at U2.34 (RXD0): now also J2.3 (P3); no longer J2.2 (P2)
- net at U2.35 (TXD0): now also J2.2 (P2); no longer J2.1 (P1)
- net EN: no longer names the net of U2.3 (EN)
- net EN: now also SW2.2; no longer J2.4 (P4)
- no-connect marks 55 -> 56
Other:
- moved on the sheet: J2
Changed lines of the file:
@@
 LIBS:ESP32-footprints-Shem-Lib
 LIBS:TexasInstruments
+LIBS:switches
 LIBS:Untitled-cache
 EELAYER 25 0
@@
 	1    0    0    -1
 $EndComp
-NoConn ~ 4150 3600
 $Comp
 L GND #PWR07
@@
 L CONN_01X06 J2
 U 1 1 5A4B1405
-P 10200 1750
-F 0 "J2" H 10200 2100 50  0000 C CNN
-F 1 "CONN_01X06" V 10300 1750 50  0000 C CNN
-F 2 "Pin_Headers:Pin_Header_Straight_1x06" H 10200 1750 50  0001 C CNN
-F 3 "" H 10200 1750 50  0001 C CNN
-	1    10200 1750
+P 10200 1650
+F 0 "J2" H 10200 2000 50  0000 C CNN
+F 1 "CONN_01X06" V 10300 1650 50  0000 C CNN
+F 2 "Pin_Headers:Pin_Header_Straight_1x06" H 10200 1650 50  0001 C CNN
+F 3 "" H 10200 1650 50  0001 C CNN
+	1    10200 1650
 	1    0    0    -1
 $EndComp
@@
 Wire Wire Line
 	9400 1600 10000 1600
-Wire Wire Line
-	10000 1700 9800 1700
-Wire Wire Line
-	9800 1700 9800 2500
-Wire Wire Line
-	9800 2500 9400 2500
-Wire Wire Line
-	10000 2000 10000 2700
-Wire Wire Line
-	10000 2700 9400 2700
-Text GLabel 10000 1800 0    60   Input ~ 0
-EN
-Text GLabel 10000 1900 0    60   Input ~ 0
+Text GLabel 10000 1700 0    60   Input ~ 0
 33
 Text GLabel 7200 1350 1    60   Input ~ 0
 33
-Text GLabel 7550 1550 0    60   Output ~ 0
-EN
 $Comp
 L GND #PWR017
@@
 Wire Wire Line
 	5900 3750 5900 4700
+$Comp
+L GND #PWR023
+U 1 1 5A51FD33
+P 10000 1900
+F 0 "#PWR023" H 10000 1650 50  0001 C CNN
+F 1 "GND" H 10000 1750 50  0000 C CNN
+F 2 "" H 10000 1900 50  0001 C CNN
+F 3 "" H 10000 1900 50  0001 C CNN
+	1    10000 1900
+	1    0    0    -1
+$EndComp
+NoConn ~ 10000 1400
+NoConn ~ 10000 1800
+Wire Wire Line
+	7550 1550 7400 1550
+Wire Wire Line
+	7400 1550 7400 2250
+Wire Wire Line
+	7400 2250 7000 2250
+$Comp
+L SW_Push SW3
+U 1 1 5A520A39
+P 9600 2500
+F 0 "SW3" H 9650 2600 50  0000 L CNN
+F 1 "SW_Push" H 9600 2440 50  0000 C CNN
+F 2 "Buttons_Switches_SMD:SW_SPST_EVQPE1" H 9600 2700 50  0001 C CNN
+F 3 "" H 9600 2700 50  0001 C CNN
+	1    9600 2500
+	1    0    0    -1
+$EndComp
+$Comp
+L GND #PWR024
+U 1 1 5A520B2E
+P 9900 2500
+F 0 "#PWR024" H 9900 2250 50  0001 C CNN
+F 1 "GND" H 9900 2350 50  0000 C CNN
+F 2 "" H 9900 2500 50  0001 C CNN
+F 3 "" H 9900 2500 50  0001 C CNN
+	1    9900 2500
+	1    0    0    -1
+$EndComp
+Wire Wire Line
+	9900 2500 9800 2500
+$Comp
+L SW_Push SW2
+U 1 1 5A520C6F
+P 6800 2250
+F 0 "SW2" H 6850 2350 50  0000 L CNN
+F 1 "SW_Push" H 6800 2190 50  0000 C CNN
+F 2 "Buttons_Switches_SMD:SW_SPST_EVQPE1" H 6800 2450 50  0001 C CNN
+F 3 "" H 6800 2450 50  0001 C CNN
+	1    6800 2250
+	1    0    0    -1
+$EndComp
+Wire Wire Line
+	6600 2250 6500 2250
+$Comp
+L GND #PWR025
+U 1 1 5A520D50
+P 6500 2250
+F 0 "#PWR025" H 6500 2000 50  0001 C CNN
+F 1 "GND" H 6500 2100 50  0000 C CNN
+F 2 "" H 6500 2250 50  0001 C CNN
+F 3 "" H 6500 2250 50  0001 C CNN
+	1    6500 2250
+	1    0    0    -1
+$EndComp
+$Comp
+L SW_Push SW1
+U 1 1 5A520EF9
+P 4350 3300
+F 0 "SW1" H 4400 3400 50  0000 L CNN
+F 1 "SW_Push" H 4350 3240 50  0000 C CNN
+F 2 "Buttons_Switches_SMD:SW_SPST_EVQPE1" H 4350 3500 50  0001 C CNN
+F 3 "" H 4350 3500 50  0001 C CNN
+	1    4350 3300
+	1    0    0    -1
+$EndComp
+$Comp
+L GND #PWR026
+U 1 1 5A520F67
+P 4650 3300
+F 0 "#PWR026" H 4650 3050 50  0001 C CNN
+F 1 "GND" H 4650 3150 50  0000 C CNN
+F 2 "" H 4650 3300 50  0001 C CNN
+F 3 "" H 4650 3300 50  0001 C CNN
+	1    4650 3300
+	1    0    0    -1
+$EndComp
+Wire Wire Line
+	4650 3300 4550 3300
+Wire Wire Line
+	4150 3300 4150 3600
 $EndSCHEMATC

Commit message: Removed an unused label
Parts:
- R11, R12: value R -> 330
- R2, R3, R4: value 330 -> 470
Connections:
- net CLR: no longer names the net of U2.31 (IO19)
- no-connect marks 56 -> 57
Changed lines of the file:
@@
 P 3900 1550
 F 0 "R2" V 3980 1550 50  0000 C CNN
-F 1 "330" V 3900 1550 50  0000 C CNN
+F 1 "470" V 3900 1550 50  0000 C CNN
 F 2 "Resistors_SMD:R_1206_HandSoldering" V 3830 1550 50  0001 C CNN
 F 3 "" H 3900 1550 50  0001 C CNN
@@
 P 3900 1950
 F 0 "R3" V 3980 1950 50  0000 C CNN
-F 1 "330" V 3900 1950 50  0000 C CNN
+F 1 "470" V 3900 1950 50  0000 C CNN
 F 2 "Resistors_SMD:R_1206_HandSoldering" V 3830 1950 50  0001 C CNN
 F 3 "" H 3900 1950 50  0001 C CNN
@@
 P 3900 2350
 F 0 "R4" V 3980 2350 50  0000 C CNN
-F 1 "330" V 3900 2350 50  0000 C CNN
+F 1 "470" V 3900 2350 50  0000 C CNN
 F 2 "Resistors_SMD:R_1206_HandSoldering" V 3830 2350 50  0001 C CNN
 F 3 "" H 3900 2350 50  0001 C CNN
@@
 	1    0    0    -1
 $EndComp
-Text GLabel 9400 2300 2    60   Input ~ 0
+Text GLabel 9400 2300 2    60   Output ~ 0
 DATA
-Text GLabel 9400 2000 2    60   Input ~ 0
+Text GLabel 9400 2000 2    60   Output ~ 0
 CLK
-Text GLabel 9400 1900 2    60   Input ~ 0
-CLR
-Text GLabel 9400 2100 2    60   Input ~ 0
+Text GLabel 9400 2100 2    60   Output ~ 0
 LATCH
-Text GLabel 9400 2200 2    60   Input ~ 0
+Text GLabel 9400 2200 2    60   Output ~ 0
 OE
 $Comp
@@
 P 6400 5600
 F 0 "R11" V 6300 5600 50  0000 C CNN
-F 1 "R" V 6400 5600 50  0000 C CNN
+F 1 "330" V 6400 5600 50  0000 C CNN
 F 2 "Resistors_SMD:R_1206_HandSoldering" V 6330 5600 50  0001 C CNN
 F 3 "" H 6400 5600 50  0001 C CNN
@@
 P 8900 5600
 F 0 "R12" V 8800 5600 50  0000 C CNN
-F 1 "R" V 8900 5600 50  0000 C CNN
+F 1 "330" V 8900 5600 50  0000 C CNN
 F 2 "Resistors_SMD:R_1206_HandSoldering" V 8830 5600 50  0001 C CNN
 F 3 "" H 8900 5600 50  0001 C CNN
@@
 Wire Wire Line
 	4150 3300 4150 3600
+NoConn ~ 9400 1900
 $EndSCHEMATC
